File: som.kicad_sch (KiCad schematic)
At the start: 228 parts, among them J1 TF, J2 Conn_Debug, J3 Conn_MP, J4 Conn_PB, J5 Conn_PA, J6 Conn_PWR, J7 Conn_IIC, U1 XC7Z010CLG400, U2 CH340E, U3 USB3300, U4 AP6212, U5 DS3231SN, U6 MT41K256M16, U7 STPMIC1, X1 32768Hz, X2 26MHz, X3 24MHz, X4 33.3MHz, X5 50MHz

Commit message: v0r2
Parts:
- removed D10, D4, D5, D6, D7, D8, D9: TVS, Resistor_SMD:R_0201_0603Metric, symbol Device:D_TVS
- removed R14: 4K7Ω, Resistor_SMD:R_0201_0603Metric, symbol Device:R
- added R21, R9: 22Ω, Resistor_SMD:R_0201_0603Metric, symbol Device:R
- added RN10: 4K7Ω, Resistor_SMD:R_Array_Convex_4x0402, symbol Device:R_Pack04
- AE1: footprint Connector_Coaxial:U.FL_Molex_MCRF_73412-0110_Vertical -> Stanlazys:U.FL_Molex_MCRF_73412-0110_Vertical
- D4: renamed from D11; footprint LED_SMD:LED_Lumex_SML-LX0404SIUPGUSB -> Stanlazys:LED_Lumex_SML-LX0404SIUPGUSB; symbol Device:LED_ABGR -> Device:LED_ARGB
- X1, X2, X3, X5: footprint Crystal:Crystal_SMD_2520-4Pin_2.5x2.0mm -> Stanlazys:Crystal_SMD_2520-4Pin_2.5x2.0mm
- renumbered D17 to D10, D18 to D11, D19 to D12, D20 to D13, D21 to D14, D22 to D15, D12 to D5, D13 to D6, D14 to D7, D15 to D8, D16 to D9, R9 to R10, R10 to R11, R11 to R12, R12 to R13, R13 to R14, R17 to R15, R15 to R17, RN10 to RN11, RN11 to RN12
Connections:
- net +3V3: now also RN10.5 (R4.2), RN10.6 (R3.2), RN10.7 (R2.2), RN10.8 (R1.2)
- net JTAG_TCK: now also RN10.3 (R3.1)
- net JTAG_TDI: now also RN10.4 (R4.1)
- net JTAG_TMS: now also RN10.2 (R2.1)
- net LED1_B: now also R17.1, U1.L19 (IO_L9P_T1_DQS_AD3P_35); no longer R15.1, U1.L20 (IO_L9N_T1_DQS_AD3N_35)
- net LED1_B_: now also D4.4 (BK), R17.2; no longer D4.2 (BK), R15.2
- net LED1_R: now also R15.1, U1.L20 (IO_L9N_T1_DQS_AD3N_35); no longer R17.1, U1.L19 (IO_L9P_T1_DQS_AD3P_35)
- net LED1_R_: now also D4.2 (RK), R15.2; no longer D4.4 (RK), R17.2
- net PL_CLK: now also R21.2; no longer X5.3 (OUT)
- net PS_CLK: now also R9.2; no longer X4.3 (OUT)
- net PS_SRST: now also RN10.1 (R1.1)
- new net PL_CLK_: R21.1, X5.3 (OUT)
- new net PS_CLK_: R9.1, X4.3 (OUT)
Other:
- note added: "L20 M20 L19 M19 Y14 J19 K19 M14 M15 M17 L15 L16 K16 J16 J14 H16"
- note removed: "L19 M20 L20 M19 Y14 J19 K19 M14 M15 M17 L15 L16 K16 J16 J14 H16"
